Commit message: #2 Fix inertia and plane parameters
Fix inertia in ball urdf and add plane parameters (restitution, contactDamping, contactStiffness). Add command wrapper for getDynamicsInfo.

File: urdf_models/ball.urdf (robot description, URDF)
Before this commit: robot simple_ball, 1 links, 0 joints
Links:
- link ball: mass 1.0 -> 0.0027; geometry collision sphere radius=0.04; visual sphere radius=0.04

Commit message: #2 Fix radius and inertia

File: urdf_models/ball.urdf (robot description, URDF)
Before this commit: robot simple_ball, 1 links, 0 joints
Links:
- link ball: geometry collision sphere radius=0.02; visual sphere radius=0.02
