Commit message: Paddle urdf changed, in order to adjust the rotation axes. Paddle get_center method adjusted, because the id of the center joint has changed.

File: paddle/paddle.urdf (robot description, URDF)
Before this commit: robot robot, 8 links, 7 joints
Joints:
- joint paddle_to_handle: child pad -> handle; origin xyz=0.18 -0.0125 0 -> xyz=0.18 0 0; parent handle -> pad
- joint x_gripper_roll: child handle -> pad

Commit message: Debug: pid plotting

File: paddle/paddle.urdf (robot description, URDF)
Before this commit: robot robot, 8 links, 7 joints
Links:
- link pad: geometry collision cylinder length=0.01 radius=0.085; visual cylinder length=0.01 radius=0.085
